File: Switch Big/Switch Big.kicad_pcb (KiCad board)
At the start: 2 copper layers, 97.2 x 128.4 mm, 23 parts, among them SW1 SW_SPDT, SW2 SW_SPDT, SW3 SW_SPDT, SW4 SW_SPDT, SW5 SW_SPDT

Commit message: Update Switch Big.kicad_pcb
Parts:
- removed kibuzzard-63947E6E: G***, kibuzzard-63947E6E
- removed kibuzzard-63947F04: G***, kibuzzard-63947F04
- added kibuzzard-6564ECD4: G***, kibuzzard-6564ECD4, F.Cu at (46.6, 141.3)
- added kibuzzard-6564ED25: G***, kibuzzard-6564ED25, F.Cu at (46.6, 143.5)
- moved kibuzzard-63972479 32.6 mm to (11.6, 138.8)
- moved SW1 2.00 mm to (103.0, 36.1)
- moved SW2 2.00 mm to (103.0, 59.1)
- moved SW3 2.00 mm to (103.0, 82.2)
- moved SW4 2.00 mm to (103.0, 105.2)
- moved SW5 2.00 mm to (103.0, 128.2)
Routing:
- net Net-(SW2-B): track 14.7 -> 16.7 mm
- net Net-(SW2-A): track 23.7 -> 21.7 mm
- net Net-(SW2-C): track 38.6 -> 37.9 mm
Other:
- outline, holes or cut-outs redrawn
