File: Switch Big/Switch Big.kicad_pcb (KiCad board)
At the start: 2 copper layers, 97.2 x 128.4 mm, 23 parts, among them SW1 SW_SPDT, SW2 SW_SPDT, SW3 SW_SPDT, SW4 SW_SPDT, SW5 SW_SPDT

Commit message: GND
Routing:
- added copper zone on B.Cu, net (none)
- added copper zone on F.Cu, net (none)
Changed lines of the file:
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@@
     (connect_pads (clearance 0.5))
     (min_thickness 0.25) (filled_areas_thickness no)
-    (fill (thermal_gap 0.5) (thermal_bridge_width 0.5))
+    (fill yes (thermal_gap 0.5) (thermal_bridge_width 0.5))
     (polygon
       (pts
@@
       )
     )
+  )
+  (zone (net 0) (net_name "") (layers "F&B.Cu") (hatch edge 0.5)
+    (priority 1)
+    (connect_pads (clearance 0.5))
+    (min_thickness 0.25) (filled_areas_thickness no)
+    (fill yes (thermal_gap 0.5) (thermal_bridge_width 0.5) (island_removal_mode 1) (island_area_min 10))
+    (polygon
+      (pts
+        (xy 66.8 21.1)
+        (xy 26.5 21.075)
+        (xy 26.5 149.5)
+        (xy 66.8 149.5)
+      )
+    )

Commit message: Fills
Parts:
- removed kibuzzard-63947E6E: G***, kibuzzard-63947E6E
- removed kibuzzard-63947F04: G***, kibuzzard-63947F04
- removed kibuzzard-63972479: G***, kibuzzard-63972479
- added kibuzzard-63663374: G***, kibuzzard-63663374, F.Cu at (92.9, 137.8)
- added kibuzzard-63663374: G***, kibuzzard-63663374, B.Cu at (46.5, 116.4)
- added kibuzzard-63663374: G***, kibuzzard-63663374, B.Cu at (102.3, 137.8)
- added kibuzzard-63729A5C: G***, kibuzzard-63729A5C, F.Cu at (97.6, 135.2)
- added kibuzzard-63729A5C: G***, kibuzzard-63729A5C, B.Cu at (97.6, 135.2)
- added kibuzzard-63729A5C: G***, kibuzzard-63729A5C, B.Cu at (41.8, 113.8)
- added kibuzzard-63920CDF: G***, kibuzzard-63920CDF, F.Cu at (93.2, 59.7)
- added kibuzzard-63920CDF: G***, kibuzzard-63920CDF, F.Cu at (93.2, 128.0)
- added kibuzzard-63920CDF: G***, kibuzzard-63920CDF, F.Cu at (93.2, 82.5)
- added kibuzzard-63920CDF: G***, kibuzzard-63920CDF, F.Cu at (93.2, 37.0)
- added kibuzzard-63920CDF: G***, kibuzzard-63920CDF, F.Cu at (93.2, 105.2)
- added kibuzzard-6564ECD4: G***, kibuzzard-6564ECD4, F.Cu at (54.0, 138.9)
- added kibuzzard-6564ED25: G***, kibuzzard-6564ED25, F.Cu at (54.0, 141.1)
- added kibuzzard-65662F15: G***, kibuzzard-65662F15, F.Cu at (42.3, 40.8)
- added kibuzzard-65662F7A: G***, kibuzzard-65662F7A, F.Cu at (42.3, 63.7)
- added kibuzzard-65662F7F: G***, kibuzzard-65662F7F, F.Cu at (42.3, 86.6)
- added kibuzzard-65662F83: G***, kibuzzard-65662F83, F.Cu at (42.3, 109.5)
- added kibuzzard-65662F89: G***, kibuzzard-65662F89, F.Cu at (42.3, 132.5)
- moved SW3 9.66 mm to (110.4, 79.8)
- moved SW4 9.66 mm to (110.4, 102.8)
- moved SW5 9.66 mm to (110.4, 125.8)
- moved SW1 9.66 mm to (110.4, 33.8)
- moved SW2 9.66 mm to (110.4, 56.8)
- moved In3 7.73 mm to (96.4, 74.8)
- moved In4 7.73 mm to (96.4, 97.8)
- moved In5 7.73 mm to (96.4, 120.8)
- moved Out10 7.73 mm to (117.9, 134.3)
- moved Out4 7.73 mm to (117.9, 65.3)
- moved Out5 7.73 mm to (117.9, 77.8)
- moved Out6 7.73 mm to (117.9, 88.3)
- moved Out7 7.73 mm to (117.9, 100.8)
- moved Out8 7.73 mm to (117.9, 111.3)
- moved Out9 7.73 mm to (117.9, 123.8)
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Routing:
- net Net-(SW4-B): track 14.7 -> 16.7 mm
- net Net-(SW3-B): track 14.7 -> 16.7 mm
- net Net-(SW2-A): track 23.7 -> 21.7 mm
- net Net-(SW1-A): track 23.7 -> 21.7 mm
- net Net-(SW5-B): track 14.7 -> 16.7 mm
- net Net-(SW5-A): track 23.7 -> 21.7 mm
- net Net-(SW4-A): track 23.7 -> 21.7 mm
- net Net-(SW3-A): track 23.7 -> 21.7 mm
- net Net-(SW2-B): track 14.7 -> 16.7 mm
- net Net-(SW1-B): track 14.7 -> 16.7 mm
- net Net-(SW1-C): track 38.9 -> 37.7 mm
- net Net-(SW4-C): track 38.0 -> 37.1 mm
- net Net-(SW2-C): track 38.6 -> 37.8 mm
- net Net-(SW5-C): track 36.3 -> 35.8 mm
Other:
- board size 97.2 x 128.4 mm -> 97.3 x 128.4 mm
- board text added: "Big Switch"
- board text added: "v0.01"
