File: Multiple/Multiple.kicad_sch (KiCad schematic)
At the start: 8 parts

Commit message: GND
Connections:
- no-connect marks 7 -> 8
Changed lines of the file:
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@@
   (no_connect (at 25.4 46.99))
   (no_connect (at 25.4 83.82))
+  (no_connect (at 25.4 73.66))
   (no_connect (at 25.4 57.15))
   (no_connect (at 25.4 104.14))

Commit message: Updates
Parts:
- added Out9: AudioJack2_SwitchT, Connector_Audio:Jack_3.5mm_QingPu_WQP-PJ398SM_Vertical_CircularHoles, symbol Connector_Audio:AudioJack2_SwitchT
Connections:
- net GND: now also Out9.S
- net at Out1.T, Out2.T, Out3.T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: now also Out9.T
- no-connect marks 8 -> 9
Other:
- moved on the sheet: Out5, Out6, Out7, Out8
