File: Switch/Switch.kicad_pcb (KiCad board)
At the start: 2 copper layers, 22.1 x 128.6 mm, 16 parts, among them SW1 SW_SPDT, SW2 SW_SPDT

Commit message: Fixed kicad issues
Parts:
- removed REF**: OSHW-Logo2_7.3x6mm_SilkScreen, Symbol:OSHW-Logo2_7.3x6mm_SilkScreen
- removed REF**: KiCad-Logo2_5mm_SilkScreen, Symbol:KiCad-Logo2_5mm_SilkScreen
- removed REF**: WEEE-Logo_4.2x6mm_SilkScreen, Symbol:WEEE-Logo_4.2x6mm_SilkScreen
- removed REF**: ESD-Logo_6.6x6mm_SilkScreen, Symbol:ESD-Logo_6.6x6mm_SilkScreen
- removed kibuzzard-63947E6E: G***, kibuzzard-63947E6E
- removed kibuzzard-63947F04: G***, kibuzzard-63947F04
- removed kibuzzard-63970E2D: G***, kibuzzard-63970E2D
- removed kibuzzard-63972479: G***, kibuzzard-63972479
- added kibuzzard-6564E20D: G***, kibuzzard-6564E20D, F.Cu at (29.0, 139.1)
- added kibuzzard-6564E26E: G***, kibuzzard-6564E26E, F.Cu at (29.0, 84.4)
- added kibuzzard-6564E2EE: G***, kibuzzard-6564E2EE, F.Cu at (29.0, 141.4)
- added kibuzzard-6564E561: G***, kibuzzard-6564E561, F.Cu at (37.5, 127.3)
- added kibuzzard-6564E561: G***, kibuzzard-6564E561, B.Cu at (32.7, 127.2)
- added kibuzzard-6564E561: G***, kibuzzard-6564E561, B.Cu at (45.1, 127.3)
- added kibuzzard-6564E629: G***, kibuzzard-6564E629, F.Cu at (44.9, 127.2)
- added kibuzzard-6564E629: G***, kibuzzard-6564E629, B.Cu at (25.4, 127.1)
- added kibuzzard-6564E629: G***, kibuzzard-6564E629, B.Cu at (37.7, 127.2)
Other:
- board size 22.1 x 128.6 mm -> 22.1 x 128.4 mm

Commit message: GND
Routing:
- added copper zone on B.Cu, net (none)
- added copper zone on F.Cu, net (none)
- added copper zone on B.Cu, net GND
- added copper zone on F.Cu, net GND
Changed lines of the file:
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@@
     (attr board_only exclude_from_pos_files exclude_from_bom)
     (fp_text reference "kibuzzard-6564E629" (at 0 4.46148 90) (layer "B.SilkS") hide
-        (effects (font (size 0 0)) (justify mirror))
+        (effects (font (size 0 0) (thickness 0.15)) (justify mirror))
     )
     (fp_text value "G***" (at 0 -4.46148 90) (layer "B.SilkS") hide
-        (effects (font (size 0 0)) (justify mirror))
+        (effects (font (size 0 0) (thickness 0.15)) (justify mirror))
     )
     (fp_poly
@@
   (segment (start 45.29 104.34) (end 45.29 138.19) (width 0.25) (layer "F.Cu") (net 12))
   (segment (start 45.29 138.19) (end 43.58 139.9) (width 0.25) (layer "F.Cu") (net 12))
+  (zone (net 0) (net_name "") (layers "F&B.Cu") (hatch edge 0.5)
+    (priority 1)
+    (connect_pads (clearance 0.5))
+    (min_thickness 0.25) (filled_areas_thickness no)
+    (fill yes (thermal_gap 0.5) (thermal_bridge_width 0.5) (island_removal_mode 1) (island_area_min 10))
+    (polygon
+      (pts
+        (xy 24.075 18.925)
+        (xy 33.9 18.95)
+        (xy 33.9 147.35)
+        (xy 24.075 147.325)
+      )
+    )
+  )
+  (zone (net 1) (net_name "GND") (layers "F&B.Cu") (hatch edge 0.5)
+    (connect_pads (clearance 0.5))
+    (min_thickness 0.25) (filled_areas_thickness no)
+    (fill yes (thermal_gap 0.5) (thermal_bridge_width 0.5))
+    (polygon
+      (pts
+        (xy 46.25 25.075)
+        (xy 36.25 25.075)
+        (xy 36.25 141.475)
+        (xy 46.25 141.475)
+      )
+    )
+  )
 )

Commit message: Fills
Parts:
- removed kibuzzard-6564E561 (x3): G***, kibuzzard-6564E561
- removed kibuzzard-6564E629 (x3): G***, kibuzzard-6564E629
- added kibuzzard-63663374: G***, kibuzzard-63663374, F.Cu at (38.0, 84.3)
- added kibuzzard-63663374: G***, kibuzzard-63663374, B.Cu at (44.7, 84.1)
- added kibuzzard-63663374: G***, kibuzzard-63663374, B.Cu at (32.4, 79.2)
- added kibuzzard-63729A5C: G***, kibuzzard-63729A5C, F.Cu at (44.8, 88.8)
- added kibuzzard-63729A5C: G***, kibuzzard-63729A5C, B.Cu at (25.4, 83.4)
- added kibuzzard-63729A5C: G***, kibuzzard-63729A5C, B.Cu at (38.0, 88.6)
- added kibuzzard-65663047: G***, kibuzzard-65663047, F.Cu at (29.1, 96.5)
- added kibuzzard-65663061: G***, kibuzzard-65663061, F.Cu at (29.0, 38.1)
Other:
- board text added: "Switch"
- board text added: "v0.01"

Commit message: Updates
Parts:
- removed the kibuzzard-63663374 at (38.0, 84.3)
- removed the kibuzzard-63663374 at (44.7, 84.1)
- removed the kibuzzard-63663374 at (32.4, 79.2)
- removed the kibuzzard-63729A5C at (44.8, 88.8)
- removed the kibuzzard-63729A5C at (25.4, 83.4)
- removed the kibuzzard-63729A5C at (38.0, 88.6)
- removed kibuzzard-6564E20D: G***, kibuzzard-6564E20D
- removed kibuzzard-6564E26E: G***, kibuzzard-6564E26E
- removed kibuzzard-6564E2EE: G***, kibuzzard-6564E2EE
- removed kibuzzard-65663047: G***, kibuzzard-65663047
- removed kibuzzard-65663061: G***, kibuzzard-65663061
- added REF**: KiCad-Logo2_5mm_SilkScreen, Symbol:KiCad-Logo2_5mm_SilkScreen, B.Cu at (95.3, 42.1)
- added REF**: ESD-Logo_6.6x6mm_SilkScreen, Symbol:ESD-Logo_6.6x6mm_SilkScreen, B.Cu at (102.7, 49.6)
- added REF**: WEEE-Logo_4.2x6mm_SilkScreen, Symbol:WEEE-Logo_4.2x6mm_SilkScreen, B.Cu at (102.7, 36.9)
- added REF**: OSHW-Logo2_7.3x6mm_SilkScreen, Symbol:OSHW-Logo2_7.3x6mm_SilkScreen, B.Cu at (103.0, 42.5)
- added kibuzzard-63663374: G***, kibuzzard-63663374, F.Cu at (72.5, 43.5)
- added kibuzzard-63663374: G***, kibuzzard-63663374, B.Cu at (81.9, 43.5)
- added kibuzzard-63729A5C: G***, kibuzzard-63729A5C, F.Cu at (77.2, 40.9)
- added kibuzzard-63729A5C: G***, kibuzzard-63729A5C, B.Cu at (77.2, 40.9)
- added kibuzzard-63920CDF: G***, kibuzzard-63920CDF, F.Cu at (128.0, 114.9)
- added kibuzzard-63920CDF: G***, kibuzzard-63920CDF, F.Cu at (70.6, 94.8)
- added kibuzzard-63948EC7: G***, kibuzzard-63948EC7, F.Cu at (101.8, 48.8)
- added kibuzzard-63948EC7: G***, kibuzzard-63948EC7, F.Cu at (101.7, 72.9)
- added kibuzzard-63948EE9: G***, kibuzzard-63948EE9, F.Cu at (96.5, 62.6)
- added kibuzzard-63948EE9: G***, kibuzzard-63948EE9, F.Cu at (96.4, 26.9)
- added kibuzzard-656B60C2: G***, kibuzzard-656B60C2, F.Cu at (99.3, 134.7)
- added kibuzzard-656B617B: G***, kibuzzard-656B617B, B.Cu at (99.3, 24.4)
- added kibuzzard-656C56A9: G***, kibuzzard-656C56A9, F.Cu at (99.4, 132.4)
- moved SW2 62.9 mm to (77.1, 53.3)
- moved In1 50.6 mm to (71.4, 67.2), turned to 90 degrees
- moved Out1 45.7 mm to (71.4, 89.4), turned to 90 degrees
- moved Out2 42.5 mm to (71.4, 99.5), turned to 90 degrees
- moved SW1 38.9 mm to (77.1, 31.5)
- moved Out4 31.3 mm to (71.4, 120.0), turned to 90 degrees
- moved In2 31.1 mm to (71.4, 77.3), turned to 90 degrees
- moved Out3 30.4 mm to (71.4, 109.8), turned to 90 degrees
Routing:
- net GND: track 125.9 -> 52.8 mm
- net Net-(SW1-A): track 19.8 -> 60.3 mm
- net Net-(SW2-A): track 19.3 -> 56.0 mm
- net Net-(SW2-C): track 44.3 -> 78.1 mm, vias 0 -> 1
- net Net-(SW1-C): track 45.8 -> 75.1 mm
- net Net-(SW1-B): track 13.1 -> 40.3 mm
- net Net-(SW2-B): track 13.4 -> 28.1 mm
Other:
- board size 22.1 x 128.4 mm -> 36.8 x 128.4 mm
- board text added: "JLCJLCJLCJLC"
