File: MultipleBuffered/MultipleBuffered.kicad_sch (KiCad schematic)
At the start: 38 parts, among them J1 Conn_02x05_Odd_Even, U1 TL074, U2 TL074, U3 TL071

Commit message: Updates
Parts:
- removed C7, C8: 100nf, Capacitor_THT:C_Disc_D5.0mm_W2.5mm_P2.50mm, symbol Device:C
- removed In2, Out5: AudioJack2_SwitchT, Connector_Audio:Jack_3.5mm_QingPu_WQP-PJ398SM_Vertical_CircularHoles, symbol Connector_Audio:AudioJack2_SwitchT
- removed R11, R12: 10r, Resistor_THT:R_Axial_DIN0207_L6.3mm_D2.5mm_P2.54mm_Vertical, symbol NanoGris-rescue:R-Device-GridsNanoV3-rescue
- removed R6: 1K, Resistor_THT:R_Axial_DIN0207_L6.3mm_D2.5mm_P2.54mm_Vertical, symbol Device:R
- removed U3: TL071, symbol Amplifier_Operational:TL071
- added H1, H2: MountingHole, MountingHole:MountingHole_3.2mm_M3, symbol Mechanical:MountingHole
- added In1: AudioJack2_SwitchT, Connector_Audio:Jack_3.5mm_QingPu_WQP-PJ398SM_Vertical_CircularHoles, symbol Connector_Audio:AudioJack2_SwitchT
- added J1, J2: Conn_01x05, Connector_PinHeader_2.54mm:PinHeader_1x05_P2.54mm_Vertical, symbol Connector_Generic:Conn_01x05
- added J3, J4: Conn_01x05, Connector_PinSocket_2.54mm:PinSocket_1x05_P2.54mm_Vertical, symbol Connector_Generic:Conn_01x05
- added J6: Conn_01x02, Connector_PinHeader_2.54mm:PinHeader_1x02_P2.54mm_Vertical, symbol Connector_Generic:Conn_01x02
- added J7: Conn_01x02, Connector_PinSocket_2.54mm:PinSocket_1x02_P2.54mm_Vertical, symbol Connector_Generic:Conn_01x02
- D1: renamed from D4; footprint (none) -> LED_THT:LED_D3.0mm
- D2: renamed from D3; footprint (none) -> LED_THT:LED_D3.0mm
- R1: renamed from R2; footprint Resistor_THT:R_Axial_DIN0207_L6.3mm_D2.5mm_P2.54mm_Vertical -> Resistor_THT:R_Axial_DIN0207_L6.3mm_D2.5mm_P7.62mm_Horizontal
- R10: value 330 -> 1K
- R11: renamed from R1; footprint Resistor_THT:R_Axial_DIN0207_L6.3mm_D2.5mm_P2.54mm_Vertical -> Resistor_THT:R_Axial_DIN0207_L6.3mm_D2.5mm_P7.62mm_Horizontal
- R2: renamed from R3; footprint Resistor_THT:R_Axial_DIN0207_L6.3mm_D2.5mm_P2.54mm_Vertical -> Resistor_THT:R_Axial_DIN0207_L6.3mm_D2.5mm_P7.62mm_Horizontal
- R3: renamed from R4; footprint Resistor_THT:R_Axial_DIN0207_L6.3mm_D2.5mm_P2.54mm_Vertical -> Resistor_THT:R_Axial_DIN0207_L6.3mm_D2.5mm_P7.62mm_Horizontal
- R4: renamed from R5; footprint Resistor_THT:R_Axial_DIN0207_L6.3mm_D2.5mm_P2.54mm_Vertical -> Resistor_THT:R_Axial_DIN0207_L6.3mm_D2.5mm_P7.62mm_Horizontal
- R5: renamed from R7; footprint Resistor_THT:R_Axial_DIN0207_L6.3mm_D2.5mm_P2.54mm_Vertical -> Resistor_THT:R_Axial_DIN0207_L6.3mm_D2.5mm_P7.62mm_Horizontal
- R6: renamed from R8; footprint Resistor_THT:R_Axial_DIN0207_L6.3mm_D2.5mm_P2.54mm_Vertical -> Resistor_THT:R_Axial_DIN0207_L6.3mm_D2.5mm_P7.62mm_Horizontal
- R7: renamed from R9; footprint Resistor_THT:R_Axial_DIN0207_L6.3mm_D2.5mm_P2.54mm_Vertical -> Resistor_THT:R_Axial_DIN0207_L6.3mm_D2.5mm_P7.62mm_Horizontal
- R8: renamed from R13; footprint Resistor_THT:R_Axial_DIN0207_L6.3mm_D2.5mm_P2.54mm_Vertical -> Resistor_THT:R_Axial_DIN0207_L6.3mm_D2.5mm_P7.62mm_Horizontal
- U1: footprint (none) -> Package_DIP:DIP-14_W7.62mm_Socket
- U3: renamed from U2; footprint (none) -> Package_DIP:DIP-14_W7.62mm_Socket
- renumbered C5 to C3, C6 to C4, C1 to C5, C2 to C6, C3 to C7, C4 to C8, D1 to D3, D2 to D4, In1 to In2, J1 to J5, Out6 to Out2, Out7 to Out3, Out2 to Out4, Out3 to Out5, Out4 to Out6
Connections:
- net +12V: now also C3.1, C7.1, D3.1 (K), U1.4 (V+), U3.4 (V+)
- net -12V: now also C4.1, C8.1, D4.2 (A), U1.11 (V-), U3.11 (V-)
- net GND: now also R10.1, In1.S, J6.1 (Pin_1), J6.2 (Pin_2), J7.1 (Pin_1), J7.2 (Pin_2)
- net at R10.2: now also In1.T, J4.1 (Pin_1); no longer D2.2 (AK)
- net at U3.10 (+), U3.12 (+), U3.3 (+)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: now also J1.1 (Pin_1)
- net at R6.2: now also J1.3 (Pin_3); no longer Out2.T
- net at R5.2: now also J1.2 (Pin_2); no longer Out1.T
- net at R4.2: now also J2.5 (Pin_5)
- net at U1.10 (+), U1.12 (+), U1.3 (+)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: now also J2.1 (Pin_1); no longer In2.T, R11.2
- net at R2.2: now also J2.3 (Pin_3); no longer Out5.T
- net at D1.2 (AK): now also J4.5 (Pin_5); no longer R8.2
- net at R1.2: now also J2.2 (Pin_2); no longer Out4.T
- net at R7.2: now also J1.4 (Pin_4); no longer Out3.T
- net at Out6.T: now also J3.4 (Pin_4); no longer R3.2
- new net: J4.3 (Pin_3), Out2.T
- new net: In2.T, J3.1 (Pin_1), R11.2
- new net: J3.3 (Pin_3), Out5.T
- new net: J3.2 (Pin_2), Out4.T
- new net: D2.2 (AK), J3.5 (Pin_5)
- new net: J4.2 (Pin_2), Out1.T
- new net: J4.4 (Pin_4), Out3.T
- new net: J1.5 (Pin_5), R8.2
- new net: J2.4 (Pin_4), R3.2
Other:
- moved on the sheet: C5, C6, D1, D2, In2, Out1, Out2, Out3, Out4, Out5, Out6, R11
